File: hardware/MillerV1/MillerV1.kicad_pcb (KiCad board)
At the start: 4 copper layers, 120 x 80 mm, 282 parts, among them IC1 TUSB1106PWR, J2 Conn_02x04_Counter_Clockwise, Q1 Q12MHz/20pF/10ppm/4P/3.2x2.5mm, U1 CCGM1A1(FBGA-324), U10 RP2040(QFN-56_7x7mm_P0.4mm), U11 TPS62A02ADRLR(SOT-563-6), U12 TPS62A02ADRLR(SOT-563-6), U13 TPS62A02ADRLR(SOT-563-6), U14 TPS62A02ADRLR(SOT-563-6), U15 TPS62A02ADRLR(SOT-563-6)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

Commit message: added graphics
Parts:
- moved G*** 0.09 mm to (179.2, 82.2)
Other:
- board text added: "GateMate Evboard V1"
