File: hardware/MillerV1/MillerV1.kicad_pcb (KiCad board)
At the start: 4 copper layers, 120 x 80 mm, 292 parts, among them IC1 TUSB1106PWR, J2 Conn_02x04_Counter_Clockwise, Q1 Q12MHz/20pF/10ppm/4P/3.2x2.5mm, U1 CCGM1A1(FBGA-324), U10 RP2040(QFN-56_7x7mm_P0.4mm), U11 TPS62A02ADRLR(SOT-563-6), U12 TPS62A02ADRLR(SOT-563-6), U13 TPS62A02ADRLR(SOT-563-6), U14 TPS62A02ADRLR(SOT-563-6), U15 TPS62A02ADRLR(SOT-563-6)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

Commit message: kleine Änderungen und GND
Connections:
- JP1 pad 3: /VGA_Red_3 -> /VGA_Blue_0
Routing:
- net /VGA_Red_2: track 31.5 -> 47.0 mm, vias 2 -> 4
Changed lines of the file:
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@@
 			(layers "*.Cu" "*.Mask")
 			(remove_unused_layers no)
-			(net "/VGA_Red_3")
+			(net "/VGA_Blue_0")
 			(pinfunction "B_3")
 			(pintype "passive")
@@
 	)
 	(segment
+		(start 120.4 87.7)
+		(end 126.3 87.7)
+		(width 1.016)
+		(layer "F.Cu")
+		(net "+2V5")
+	)
+	(segment
 		(start 125.3 112.3)
 		(end 125.3 112.7)
@@
 	)
 	(segment
-		(start 126.3 87.7)
-		(end 120.4 87.7)
-		(width 0.762)
-		(layer "In1.Cu")
-		(net "+2V5")
-	)
-	(segment
 		(start 208.8 64.9)
 		(end 208.8 64.3)
@@
 	)
 	(segment
-		(start 130.312122 89.22636)
-		(end 141.919997 89.22636)
+		(start 141.919997 89.22636)
+		(end 142.469836 89.776199)
 		(width 0.127)
 		(layer "F.Cu")
@@
 	)
 	(segment
-		(start 155.6 91.2)
-		(end 155.2 90.8)
+		(start 125.5 86)
+		(end 127.085762 86)
 		(width 0.127)
 		(layer "F.Cu")
@@
 	)
 	(segment
-		(start 141.919997 89.22636)
-		(end 142.469836 89.776199)
+		(start 127.085762 86)
+		(end 130.312122 89.22636)
+		(width 0.127)
+		(layer "F.Cu")
+		(net "/VGA_Red_2")
+	)
+	(segment
+		(start 155.6 91.2)
+		(end 155.2 90.8)
 		(width 0.127)
 		(layer "F.Cu")
@@
 	)
 	(segment
-		(start 127.112122 86.02636)
-		(end 130.312122 89.22636)
+		(start 111.624 86)
+		(end 115 86)
+		(width 0.254)
+		(layer "F.Cu")
+		(net "/VGA_Red_2")
+	)
+	(segment
+		(start 130.312122 89.22636)
+		(end 141.919997 89.22636)
 		(width 0.127)
 		(layer "F.Cu")
@@
 	)
 	(via
+		(at 125.5 86)
+		(size 0.45)
+		(drill 0.3)
+		(layers "F.Cu" "B.Cu")
+		(net "/VGA_Red_2")
+	)
+	(via
 		(at 142.9 89.776199)
 		(size 0.45)
@@
 	)
 	(via
+		(at 115 86)
+		(size 0.45)
+		(drill 0.3)
+		(layers "F.Cu" "B.Cu")
+		(net "/VGA_Red_2")
+	)
+	(via
 		(at 155.2 90.8)
 		(size 0.45)
@@
 	)
 	(segment
+		(start 115 86)
+		(end 125.5 86)
+		(width 0.254)
+		(layer "B.Cu")
+		(net "/VGA_Red_2")
+	)
+	(segment
 		(start 143.476199 89.2)
 		(end 142.9 89.776199)
@@
 	)
 	(zone
-		(net "/VGA_Red_2")
-		(layer "F.Cu")
-		(hatch edge 0.5)
-		(priority 30696)
-		(attr
-			(teardrop
-				(type padvia)
-			)
-		)
-		(connect_pads yes
-			(clearance 0)
-		)
-		(min_thickness 0.0254)
-		(fill yes
-			(island_removal_mode 1)
-		)
-		(polygon
-			(pts
-				(xy 142.500711 89.717272) (xy 142.410909 89.807074) (xy 142.813896 89.984072) (xy 142.900707 89.776906)
-				(xy 142.813896 89.568326)
-			)
-		)
-	)
-	(zone
 		(net "/+1V1")
 		(layer "F.Cu")
@@
 			)
 		)
-	)
-	(zone
-		(net "/VGA_Red_2")
-		(layer "B.Cu")
-		(hatch edge 0.5)
-		(priority 30229)
-		(attr
-			(teardrop
-				(type padvia)
-			)
-		)
-		(connect_pads yes
-			(clearance 0)
-		)
-		(min_thickness 0.0254)
-		(fill yes
-			(island_removal_mode 1)
-		)
-		(polygon
-			(pts
-				(xy 143.263099 89.502903) (xy 143.173296 89.4131) (xy 142.813896 89.568326) (xy 142.899293 89.776906)
-				(xy 143.107873 89.862303)
-			)
-		)
