File: hardware/MillerV1/MillerV1.kicad_pcb (KiCad board)
At the start: 4 copper layers, 120 x 80 mm, 296 parts, among them IC1 TUSB1106PWR, J2 Conn_02x04_Counter_Clockwise, Q1 Q12MHz/20pF/10ppm/4P/3.2x2.5mm, U1 CCGM1A1(FBGA-324), U10 RP2040(QFN-56_7x7mm_P0.4mm), U11 TPS62A02ADRLR(SOT-563-6), U12 TPS62A02ADRLR(SOT-563-6), U13 TPS62A02ADRLR(SOT-563-6), U14 TPS62A02ADRLR(SOT-563-6), U15 TPS62A02ADRLR(SOT-563-6)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

Commit message: solved some DRC issues
Parts:
- removed FID1, FID2, FID3, FID7, FID8, FID9: Fiducial, OLIMEX_Other-FP:Fiducial1x3
- removed FID10, FID11, FID12, FID4, FID5, FID6: Fiducial, OLIMEX_Other-FP:Fiducial1x3_Paste
- MH1, MH2, MH3, MH4: value Mounting_Hole_NPTH -> MountingHole_Pad
Connections:
- MH1 pad 1: (no net) -> GND
- MH2 pad 1: (no net) -> GND
- MH3 pad 1: (no net) -> GND
- MH4 pad 1: (no net) -> GND
- PWR_LED1 pad 2: +5V_USB -> Net-(D3-A)
Routing:
- net Net-(D3-A): track 14.5 -> 44.0 mm
- net +5V_USB: track 1137.2 -> 1107.7 mm
- net GND: track 3148.5 -> 3146.9 mm
Other:
- board text added: "b1"
- board text added: "b2"
- board text added: "rp.boot"
- board text added: "rp.rst"
