File: hardware/MillerV1/MillerV1.kicad_sch (KiCad schematic)
At the start: 293 parts, among them IC1 TUSB1106PWR, J2 Conn_02x04_Counter_Clockwise, Q1 Q12MHz/20pF/10ppm/4P/3.2x2.5mm, U1 CCGM1A1(FBGA-324), U10 RP2040(QFN-56_7x7mm_P0.4mm), U11 TPS62A02ADRLR(SOT-563-6), U12 TPS62A02ADRLR(SOT-563-6), U13 TPS62A02ADRLR(SOT-563-6), U14 TPS62A02ADRLR(SOT-563-6), U15 TPS62A02ADRLR(SOT-563-6)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

Commit message: Update PCB footprints and USB power nets
Modify MillerV1.kicad_pcb: fix USB power net assignments and clean up footprints. Several USB VBUS pads were retargeted from +5V_USB (and +5V_USB_2) to the correct nets (Net-(D3-A) or +5V_USB). Added new footprints: LED SMD 0603 (D2), Diode SMC B340 (D3) wired between +5V_USB and Net-(D3-A), and a 3-pad SMD solder jumper (JP1). Removed/updated some duplicated/new resistor footprint definitions and adjusted multiple footprint positions, rotations, UUIDs and pad properties to match the updated layout.
Parts:
- added D2: LED/RED/0603, LED_SMD:LED_0603_1608Metric, symbol Device:LED
- added D3: B340, Diode_SMD:D_SMC, symbol Diode:B340
- JP1: footprint Connector_PinHeader_2.54mm:PinHeader_1x03_P2.54mm_Vertical -> Jumper:SolderJumper-3_P1.3mm_Open_RoundedPad1.0x1.5mm_NumberLabels
- R35: value 10k -> 2.2k
Connections:
- net +5V_USB_2 is gone; now on net +5V_USB: C129.1, USB-C2.A4 (VBUS), USB-C2.A9 (VBUS), USB-C2.B4 (VBUS), USB-C2.B9 (VBUS)
- net +1V8: no longer C131.1, IC1.9 (V_C_C_(_I_/O_)), R35.1
- net +2V5: now also JP1.3 (B)
- net +5V_USB: now also D2.2 (A), D3.1 (K); no longer USB-C1.A4 (VBUS), USB-C1.A9 (VBUS), USB-C1.B4 (VBUS), USB-C1.B9 (VBUS)
- net GND: now also R35.2
- net USB_2_D+: now also IC1.1 (VPU(3.3)), R33.1, R34.1, R34.2
- net USB_2_D-: now also R33.2
- net VGA_Blue_0: no longer JP1.3 (B)
- net VGA_Blue_1: now also IC1.7 (SUSPND)
- net VGA_Blue_2: now also IC1.6 (VM)
- net VGA_Blue_3: now also IC1.5 (VP)
- net VGA_Green_0: no longer IC1.10 (SPEED), R35.2
- net VGA_Green_1: no longer IC1.7 (SUSPND)
- net VGA_Green_2: now also IC1.3 (~{OE}); no longer IC1.4 (RCV)
- net VGA_Green_3: now also IC1.4 (RCV); no longer IC1.14 (VMO)
- net VGA_Red_0: no longer IC1.13 (VPO)
- net VGA_Red_1: no longer IC1.5 (VP)
- net VGA_Red_2: no longer IC1.6 (VM)
- net VM: now also IC1.2 (SO_FTCO_N)
- net at IC1.12 (D+), R32.2: no longer R34.1
- net at IC1.11 (D-), R30.2: no longer R33.1
- net at JP1.2 (C): now also C131.1, IC1.9 (V_C_C_(_I_/O_)); no longer IC1.3 (~{OE})
- new net: D3.2 (A), USB-C1.A4 (VBUS), USB-C1.A9 (VBUS), USB-C1.B4 (VBUS), USB-C1.B9 (VBUS)
- new net: D2.1 (K), R35.1
Other:
- moved on the sheet: +5V_USB1, C129, C130, C131, IC1, JP1, R30, R32, R33, R34, R80, R81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

Commit message: sollte soweit fertig sein
Connections:
- net USB_2_D+: no longer IC1.1 (VPU(3.3)), R33.1, R34.1
- net VGA_Red_2: now also IC1.13 (VPO)
- net VGA_Red_3: now also IC1.10 (SPEED)
- net VPO: now also IC1.14 (VMO)
- new net VPU(3.3): IC1.1 (VPU(3.3)), R33.1, R34.1
Changed lines of the file:
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@@
 	(text "USB Diff. Pair\nZdiff=90 Ohms!"
 		(exclude_from_sim no)
-		(at 631.19 52.07 0)
+		(at 628.65 50.8 0)
 		(effects
 			(font
@@
 	(wire
 		(pts
-			(xy 655.32 53.34) (xy 647.7 53.34)
-		)
-		(stroke
-			(width 0)
-			(type default)
-		)
-	)
-	(wire
-		(pts
 			(xy 203.2 93.98) (xy 215.9 93.98)
 		)
@@
 		)
 	)
+	(label "VGA_Red_2"
+		(at 739.14 44.45 0)
+		(effects
+			(font
+				(size 0.762 0.762)
+				(thickness 0.3048)
+				(bold yes)
+			)
+			(justify left bottom)
+		)
+	)
 	(label "SER_TX_P"
 		(at 369.57 375.92 0)
@@
 		)
 	)
+	(label "VPO"
+		(at 739.14 46.99 0)
+		(effects
+			(font
+				(size 0.762 0.762)
+				(thickness 0.3048)
+				(bold yes)
+			)
+			(justify left bottom)
+		)
+	)
 	(label "{slash}CFG_FAILED"
 		(at 165.1 180.34 0)
@@
 				(thickness 0.3048)
 				(bold yes)
+			)
+			(justify left bottom)
+		)
+	)
+	(label "VGA_Red_3"
+		(at 739.14 59.69 0)
+		(effects
+			(font
+				(size 0.762 0.762)
+				(thickness 0.3048)
+				(bold yes)

Commit message: solved some DRC issues
Parts:
- removed FID1, FID2, FID3, FID7, FID8, FID9: Fiducial, OLIMEX_Other-FP:Fiducial1x3, symbol OLIMEX_OTHER:Fiducial
- removed FID10, FID11, FID12, FID4, FID5, FID6: Fiducial, OLIMEX_Other-FP:Fiducial1x3_Paste, symbol OLIMEX_OTHER:Fiducial
- removed MH1, MH2, MH3, MH4: Mounting_Hole_NPTH, MountingHole:MountingHole_3.2mm_M3_Pad_Via, symbol OLIMEX_OTHER:Mounting_Hole_NPTH
- added MH1, MH2, MH3, MH4: MountingHole_Pad, MountingHole:MountingHole_3.2mm_M3_Pad_Via, symbol Mechanical:MountingHole_Pad
Connections:
- net +5V_USB: no longer PWR_LED1.2 (A)
- net GND: now also MH1.1, MH2.1, MH3.1, MH4.1
- net at D3.2 (A), USB-C1.A4 (VBUS), USB-C1.A9 (VBUS)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: now also PWR_LED1.2 (A)
Other:
- note removed: "Fiducials"
- moved on the sheet: PWR_LED1, R76

Commit message: minor changes
Connections:
- net ISO_AS1: no longer J2.8 (Pin_8), U6.14 (B6)
- new net ISO_AS2: J2.8 (Pin_8), U6.14 (B6)
Changed lines of the file:
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@@
 		)
 	)
-	(label "ISO_AS1"
+	(label "ISO_AS2"
 		(at 627.38 201.93 0)
 		(effects
@@
 		)
 	)
-	(label "ISO_AS1"
+	(label "ISO_AS2"
 		(at 654.05 213.36 180)
 		(effects
